Commit message: feat: 更新 L10 右手模型到官方 SDK 新版本
替换模型文件（STL/URDF/MuJoCo XML）为官方 LinkerHand SDK 最新版本，
使用解剖学命名（thumb_cmc_roll, index_pip 等）替代旧的数字命名。

- 旧 26 STL 替换为新 21 STL（移除 fixed joint 对应的 mesh）
- URDF 从 25 关节（20 revolute + 5 fixed）精简为 20 revolute
- MuJoCo XML 从新 URDF 自动转换并补充执行器和仿真配置
- FK/IK 运动链数据从新模型重新提取
- DOF 范围同步为官方 SDK 映射（侧摆 DOF 6/7/8 范围和方向修正）

File: l10_right_hand_essential/linker_hand_description/linker_hand_description/urdf/L10/linker_hand_l10_right/linker_hand_l10_right.urdf (robot description, URDF)
Before this commit: robot linker_hand_l10_right, 26 links, 25 joints
Links:
- removed link index_link0
- removed link index_link1
- removed link index_link2
- removed link index_link3
- removed link index_link4
- removed link little_link0
- removed link little_link1
- removed link little_link2
- removed link little_link3
- removed link little_link4
- removed link middle_link0
- removed link middle_link1
- removed link middle_link2
- removed link middle_link3
- removed link ring_link0
- removed link ring_link1
- removed link ring_link2
- removed link ring_link3
- removed link ring_link4
- removed link thumb_link0
- removed link thumb_link1
- removed link thumb_link2
- removed link thumb_link3
- removed link thumb_link4
- removed link thumb_link5
- added link index_distal, mass 0.00314458657125681; collision mesh filename=package://linker_hand_description/urdf/L10/linker_hand_l10_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; visual mesh filename=package://linker_hand_description/urdf/L10/linker_hand_l10_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
- added link index_metacarpals, mass 0.00903700347459462; collision mesh filename=package://linker_hand_description/urdf/L10/linker_hand_l10_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; visual mesh filename=package://linker_hand_description/urdf/L10/linker_hand_l10_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
- added link index_middle, mass 0.00283043635595588; collision mesh filename=package://linker_hand_description/urdf/L10/linker_hand_l10_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; visual mesh filename=package://linker_hand_description/urdf/L10/linker_hand_l10_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
- added link index_proximal, mass 0.00654982479821771; collision mesh filename=package://linker_hand_description/urdf/L10/linker_hand_l10_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; visual mesh filename=package://linker_hand_description/urdf/L10/linker_hand_l10_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
- added link middle_distal, mass 0.0031445865911477; collision mesh filename=package://linker_hand_description/urdf/L10/linker_hand_l10_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; visual mesh filename=package://linker_hand_description/urdf/L10/linker_hand_l10_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
- added link middle_middle, mass 0.00283043635504843; collision mesh filename=package://linker_hand_description/urdf/L10/linker_hand_l10_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; visual mesh filename=package://linker_hand_description/urdf/L10/linker_hand_l10_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
- added link middle_proximal, mass 0.00654982478226948; collision mesh filename=package://linker_hand_description/urdf/L10/linker_hand_l10_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; visual mesh filename=package://linker_hand_description/urdf/L10/linker_hand_l10_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
- added link pinky_distal, mass 0.0031445864920905; collision mesh filename=package://linker_hand_description/urdf/L10/linker_hand_l10_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; visual mesh filename=package://linker_hand_description/urdf/L10/linker_hand_l10_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
- added link pinky_metacarpals, mass 0.00903700347459465; collision mesh filename=package://linker_hand_description/urdf/L10/linker_hand_l10_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; visual mesh filename=package://linker_hand_description/urdf/L10/linker_hand_l10_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
- added link pinky_middle, mass 0.00283043635595589; collision mesh filename=package://linker_hand_description/urdf/L10/linker_hand_l10_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; visual mesh filename=package://linker_hand_description/urdf/L10/linker_hand_l10_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
- added link pinky_proximal, mass 0.00654982918810593; collision mesh filename=package://linker_hand_description/urdf/L10/linker_hand_l10_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; visual mesh filename=package://linker_hand_description/urdf/L10/linker_hand_l10_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
- added link ring_distal, mass 0.0031445863941225; collision mesh filename=package://linker_hand_description/urdf/L10/linker_hand_l10_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; visual mesh filename=package://linker_hand_description/urdf/L10/linker_hand_l10_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
- added link ring_metacarpals, mass 0.00903700347459463; collision mesh filename=package://linker_hand_description/urdf/L10/linker_hand_l10_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; visual mesh filename=package://linker_hand_description/urdf/L10/linker_hand_l10_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
- added link ring_middle, mass 0.00283043628669241; collision mesh filename=package://linker_hand_description/urdf/L10/linker_hand_l10_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; visual mesh filename=package://linker_hand_description/urdf/L10/linker_hand_l10_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
- added link ring_proximal, mass 0.00654982867950541; collision mesh filename=package://linker_hand_description/urdf/L10/linker_hand_l10_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; visual mesh filename=package://linker_hand_description/urdf/L10/linker_hand_l10_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
- added link thumb_distal, mass 0.00512933613321634; collision mesh filename=package://linker_hand_description/urdf/L10/linker_hand_l10_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; visual mesh filename=package://linker_hand_description/urdf/L10/linker_hand_l10_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
- added link thumb_metacarpals, mass 0.0152011697874328; collision mesh filename=package://linker_hand_description/urdf/L10/linker_hand_l10_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; visual mesh filename=package://linker_hand_description/urdf/L10/linker_hand_l10_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
- added link thumb_metacarpals_base1, mass 0.0084581719416891; collision mesh filename=package://linker_hand_description/urdf/L10/linker_hand_l10_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; visual mesh filename=package://linker_hand_description/urdf/L10/linker_hand_l10_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
- added link thumb_metacarpals_base2, mass 0.00582710536801184; collision mesh filename=package://linker_hand_description/urdf/L10/linker_hand_l10_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; visual mesh filename=package://linker_hand_description/urdf/L10/linker_hand_l10_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
- added link thumb_proximal, mass 0.00662230120907192; collision mesh filename=package://linker_hand_description/urdf/L10/linker_hand_l10_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; visual mesh filename=package://linker_hand_description/urdf/L10/linker_hand_l10_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
- link base_link: mass 0.0813387471555535 -> 0.10884427610512
Joints:
- removed joint index_joint0
- removed joint index_joint1
- removed joint index_joint2
- removed joint index_joint3
- removed joint index_joint4
- removed joint little_joint0
- removed joint little_joint1
- removed joint little_joint2
- removed joint little_joint3
- removed joint little_joint4
- removed joint middle_joint0
- removed joint middle_joint1
- removed joint middle_joint2
- removed joint middle_joint3
- removed joint ring_joint0
- removed joint ring_joint1
- removed joint ring_joint2
- removed joint ring_joint3
- removed joint ring_joint4
- removed joint thumb_joint0
- removed joint thumb_joint1
- removed joint thumb_joint2
- removed joint thumb_joint3
- removed joint thumb_joint4
- removed joint thumb_joint5
- added joint index_dip: type revolute, parent index_middle, child index_distal, origin xyz=-0.0054686 0 0.025665 rpy=0 0 0, axis 0 1 0, limit lower=0 upper=1.8317 effort=100 velocity=1
- added joint index_mcp_pitch: type revolute, parent index_metacarpals, child index_proximal, origin xyz=0.0020763 0 0.015294 rpy=0 0 0, axis 0 1 0, limit lower=0 upper=1.3607 effort=100 velocity=1
- added joint index_mcp_roll: type revolute, parent base_link, child index_metacarpals, origin xyz=-0.0021643 0.026654 0.13253 rpy=0 0 0, axis -0.99996 0 0.0087265, limit lower=0 upper=0.2181 effort=100 velocity=1
- added joint index_pip: type revolute, parent index_proximal, child index_middle, origin xyz=-0.0013807 0 0.035624 rpy=0 0 0, axis 0 1 0, limit lower=0 upper=1.8317 effort=100 velocity=1
- added joint middle_dip: type revolute, parent middle_middle, child middle_distal, origin xyz=-0.0055098 0 0.025656 rpy=0 0 0, axis 0 1 0, limit lower=0 upper=0.628 effort=100 velocity=1
- added joint middle_mcp_pitch: type revolute, parent base_link, child middle_proximal, origin xyz=-0.0021316 0.0076542 0.15281 rpy=0 0 0, axis 0 1 0, limit lower=0 upper=1.3607 effort=100 velocity=1
- added joint middle_pip: type revolute, parent middle_proximal, child middle_middle, origin xyz=-0.001397 0 0.035623 rpy=0 0 0, axis 0 1 0, limit lower=0 upper=1.8317 effort=100 velocity=1
- added joint pinky_dip: type revolute, parent pinky_middle, child pinky_distal, origin xyz=-0.0054686 0 0.025665 rpy=0 0 0, axis 0 1 0, limit lower=0 upper=0.628 effort=100 velocity=1
- added joint pinky_mcp_pitch: type revolute, parent pinky_metacarpals, child pinky_proximal, origin xyz=0.0020763 0 0.015294 rpy=0 0 0, axis 0 1 0, limit lower=0 upper=1.3607 effort=100 velocity=1
- added joint pinky_mcp_roll: type revolute, parent base_link, child pinky_metacarpals, origin xyz=-0.00012074 -0.030346 0.12755 rpy=0 0 0, axis 0.99996 0 0.0087265, limit lower=0 upper=0.3489 effort=100 velocity=1
- added joint pinky_pip: type revolute, parent pinky_proximal, child pinky_middle, origin xyz=-0.0013807 0 0.035624 rpy=0 0 0, axis 0 1 0, limit lower=0 upper=1.8317 effort=100 velocity=1
- added joint ring_dip: type revolute, parent ring_middle, child ring_distal, origin xyz=-0.0054686 0 0.025665 rpy=0 0 0, axis 0 1 0, limit lower=0 upper=0.628 effort=100 velocity=1
- added joint ring_mcp_pitch: type revolute, parent ring_metacarpals, child ring_proximal, origin xyz=0.0020763 0 0.015294 rpy=0 0 0, axis 0 1 0, limit lower=0 upper=1.3607 effort=100 velocity=1
- added joint ring_mcp_roll: type revolute, parent base_link, child ring_metacarpals, origin xyz=-0.0021643 -0.011346 0.13253 rpy=0 0 0, axis 0.99996 0 0.0087265, limit lower=0 upper=0.2181 effort=100 velocity=1
- added joint ring_pip: type revolute, parent ring_proximal, child ring_middle, origin xyz=-0.0013807 0 0.035624 rpy=0 0 0, axis 0 1 0, limit lower=0 upper=1.8317 effort=100 velocity=1
- added joint thumb_cmc_pitch: type revolute, parent thumb_metacarpals_base2, child thumb_metacarpals, origin xyz=0.0046051 0.014383 -0.0051478 rpy=0.16356 -1.1191 -2.0038, axis 0 1 0, limit lower=0 upper=0.5146 effort=100 velocity=1
- added joint thumb_cmc_roll: type revolute, parent base_link, child thumb_metacarpals_base1, origin xyz=-0.013419 0.012551 0.060602 rpy=0 0 0, axis 0.99996 0 -0.0087265, limit lower=0 upper=1.1339 effort=100 velocity=1
- added joint thumb_cmc_yaw: type revolute, parent thumb_metacarpals_base1, child thumb_metacarpals_base2, origin xyz=0.035797 -0.00065879 0.00045944 rpy=0 0 0, axis 0.008517 -0.21782 -0.97595, limit lower=0 upper=1.9189 effort=100 velocity=0
- added joint thumb_ip: type revolute, parent thumb_proximal, child thumb_distal, origin xyz=-0.00017064 0 0.038665 rpy=0 0 0, axis 0 1 0, limit lower=0 upper=0.7763 effort=100 velocity=1
- added joint thumb_mcp: type revolute, parent thumb_metacarpals, child thumb_proximal, origin xyz=0.0061722 0 0.047968 rpy=0 0 0, axis 0 1 0, limit lower=0 upper=0.7152 effort=100 velocity=1
